File: SSD_XX_200_LPDRM.kicad_sch (KiCad schematic)
At the start: 0 parts

Commit message: Schematic Update-1.1
Other:
- sheet B2B and Peripheral Connectors renamed Backplane and Peripheral Connectors
Changed lines of the file:
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@@
 (kicad_sch
-	(version 20250114)
+	(version 20260306)
 	(generator "eeschema")
-	(generator_version "9.0")
+	(generator_version "10.0")
 	(paper "A4")
 	(title_block
@@
 		)
 		(fill
-			(color 0 0 0 0.0000)
+			(color 0 0 0 0)
 		)
 		(property "Sheetname" "Control Switches"
 			(at 128.27 47.5484 0)
+			(show_name no)
+			(do_not_autoplace no)
 			(effects
 				(font
@@
 		(property "Sheetfile" "Subsheets/Control Switches.kicad_sch"
 			(at 128.27 76.7846 0)
+			(show_name no)
+			(do_not_autoplace no)
 			(effects
 				(font
@@
 		)
 		(fill
-			(color 0 0 0 0.0000)
+			(color 0 0 0 0)
 		)
 		(property "Sheetname" "ADC"
 			(at 189.23 47.5484 0)
+			(show_name no)
+			(do_not_autoplace no)
 			(effects
 				(font
@@
 		(property "Sheetfile" "Subsheets/ADC.kicad_sch"
 			(at 189.23 76.7846 0)
+			(show_name no)
+			(do_not_autoplace no)
 			(effects
 				(font
@@
 		)
 		(fill
-			(color 0 0 0 0.0000)
+			(color 0 0 0 0)
 		)
 		(property "Sheetname" "Power Section"
 			(at 67.31 47.5484 0)
+			(show_name no)
+			(do_not_autoplace no)
 			(effects
 				(font
@@
 		(property "Sheetfile" "Subsheets/Power Section.kicad_sch"
 			(at 67.31 76.7846 0)
+			(show_name no)
+			(do_not_autoplace no)
 			(effects
 				(font
@@
 		)
 		(fill
-			(color 0 0 0 0.0000)
+			(color 0 0 0 0)
 		)
 		(property "Sheetname" "GPIO Expanders"
 			(at 67.31 85.6484 0)
+			(show_name no)
+			(do_not_autoplace no)
 			(effects
 				(font
@@
 		(property "Sheetfile" "Subshhets/GPIO Expanders.kicad_sch"
 			(at 67.31 114.8846 0)
+			(show_name no)
+			(do_not_autoplace no)
 			(effects
 				(font
@@
 		)
 		(fill
-			(color 0 0 0 0.0000)
-		)
-		(property "Sheetname" "B2B and Peripheral Connectors"
+			(color 0 0 0 0)
+		)
+		(property "Sheetname" "Backplane and Peripheral Connectors"
 			(at 128.27 86.9184 0)
+			(show_name no)
+			(do_not_autoplace no)
 			(effects
 				(font
@@
 		(property "Sheetfile" "Subsheets/B2B and Peripheral Connectors.kicad_sch"
 			(at 128.27 116.1546 0)
+			(show_name no)
+			(do_not_autoplace no)
 			(effects
 				(font
@@
 		)
 		(fill
-			(color 0 0 0 0.0000)
+			(color 0 0 0 0)
 		)
 		(property "Sheetname" "Misc"
 			(at 189.23 86.9184 0)
+			(show_name no)
+			(do_not_autoplace no)
 			(effects
 				(font
@@
 		(property "Sheetfile" "Subsheets/Misc.kicad_sch"
 			(at 189.23 116.1546 0)
-			(effects
-				(font
+			(show_name no)
+			(do_not_autoplace no)
+			(effects
+				(font
