File: Subsheets/12V_HPBM.kicad_sch (KiCad schematic)
At the start: 7 parts

Commit message: Schematic Update-1.1
Parts:
- removed C1, C2: C, symbol Device:C
- removed R21: 10k_0.0625W_0402, symbol Device:R_Small_US
- added Q37: BSS123NH6327XTSA1, SOT95P240X110-3N, symbol BSS123NH6327XTSA1:BSS123NH6327XTSA1
- added R148: 0R_0.063W_0402, Pixxel_Resistors:RES0402, symbol Device:R_Small_US
- added R44: 10k_0.0625W_0603, Pixxel_Resistors:RES0603, symbol Device:R_Small_US
- added R745: 100k_0.0625W_0402, Pixxel_Resistors:RES0402, symbol Device:R_Small_US
- added U62: (no value), symbol HVSM_LVSM_v9:HVSM
- R24: value 10k_0.0625W_0402 -> 10k_0.0625W_0603; footprint (none) -> Pixxel_Resistors:RES0603; Manufacturer Name (none) -> Vishay Dale; Manufacturer Part Number (none) -> TNPW060310K0BEEA; Price(INR) (none) -> 24.57; Temp_max (C) (none) -> 175; Temp_min (C) (none) -> -55; Vendor (none) -> Digikey; Vendor Part Number (none) -> TNP10.0KAATR-ND
- U21: value ~ -> (none)
Connections:
- net 5V: now also R148.2; no longer U21.5 (Vext)
- net BUCK_EN: now also Q37.1 (G), R44.1; no longer U21.1 (EN)
- net BUCK_IN: now also R745.2
- net GND: now also Q37.2 (S), R44.2
- new net: Q37.3 (D), R745.1, U21.1 (EN)
- new net: R148.1, U21.5 (Vext)
Other:
- moved on the sheet: TP1
