File: Subsheets/Control Switches.kicad_sch (KiCad schematic)
At the start: 240 parts

Commit message: Schematic Update-1.1
Parts:
- removed JP1, JP10, JP100, JP101, JP102, JP103, JP104, JP105, JP106, JP107, JP108, JP109, JP11, JP110, JP111, JP112, JP113, JP114, JP115, JP116, JP117, JP118, JP119, JP12, JP120, JP13, JP14, JP15, JP16, JP17, JP18, JP19, JP2, JP20, JP21, JP22, JP23, JP24, JP25, JP26, JP27, JP28, JP29, JP3, JP30, JP31, JP32, JP33, JP34, JP35, JP36, JP37, JP38, JP39, JP4, JP40, JP41, JP42, JP43, JP44, JP45, JP46, JP47, JP48, JP49, JP5, JP50, JP51, JP52, JP53, JP54, JP55, JP56, JP57, JP58, JP59, JP6, JP60, JP61, JP62, JP63, JP64, JP65, JP66, JP67, JP68, JP69, JP7, JP70, JP71, JP72, JP73, JP74, JP75, JP76, JP77, JP78, JP79, JP8, JP80, JP81, JP82, JP83, JP84, JP85, JP86, JP87, JP88, JP89, JP9, JP90, JP91, JP92, JP93, JP94, JP95, JP96, JP97, JP98, JP99: SolderJumper_2_Open, symbol Jumper:SolderJumper_2_Open
- removed R1, R10, R100, R101, R102, R11, R12, R13, R14, R15, R16, R17, R18, R19, R2, R20, R22, R23, R26, R27, R3, R30, R31, R37, R38, R4, R41, R42, R45, R46, R5, R51, R52, R53, R54, R55, R56, R57, R58, R59, R6, R60, R61, R62, R63, R64, R65, R66, R67, R68, R69, R7, R70, R75, R76, R77, R78, R79, R8, R80, R81, R82, R83, R84, R85, R86, R87, R88, R89, R9, R90, R91, R92, R93, R94, R95, R96, R97, R98, R99: 10k_0.0625W_0402, symbol Device:R_Small_US
- removed U1, U10, U11, U12, U13, U14, U15, U16, U17, U18, U19, U2, U20, U29, U3, U30, U31, U32, U33, U34, U35, U36, U37, U38, U39, U4, U40, U41, U42, U43, U44, U45, U46, U47, U48, U5, U6, U7, U8, U9: ~, symbol HVSM_LVSM_v9:LVSM
Other:
- added sheet Switch Main (Switch Main.kicad_sch)
- added sheet Switch Redundant (Switch Redundant.kicad_sch)
