File: Subsheets/LPBM.kicad_sch (KiCad schematic)
At the start: 7 parts

Commit message: Schematic Update-1.1
Parts:
- removed TP9: TestPoint, symbol Connector:TestPoint
- added R741, R743: 100k_0.0625W_0402, Pixxel_Resistors:RES0402, symbol Device:R_Small_US
- R33, R34, R35: now not fitted
- U24: value ~ -> (none)
Connections:
- net 3V3_BUCK_OUT: now also R741.2, R743.2
- net 3V3_BUCK_PG: now also R743.1
- net 5V_BUCK_PG: now also R741.1
- net 1V8_BUCK_EN: no longer names the net of R33.1
- net 1V8_BUCK_EN: no longer U24.3 (EN_1V8)
- net 1V8_BUCK_OUT: no longer names the net of U24.6 (Pout_1V8)
- net 1V8_BUCK_PG: no longer names the net of U24.9 (PG_1V8)
- net 1V8_BUCK_VMON: no longer names the net of U24.12 (Vsense_1V8)
- no-connect marks 0 -> 4
Other:
- note removed: "1v8 should be left unconnected?"
