File: Subsheets/LPBM_RED.kicad_sch (KiCad schematic)
At the start: 0 parts

Commit message: Schematic Update-1.1
Parts:
- added U8: ~, symbol Non-Isolated-Buck-Module_v9:LPBM_tri_rail
Other:
- title: (none) -> SSD_XX_200_LPDRM
Changed lines of the file:
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@@
 	(generator_version "9.0")
 	(paper "A4")
+	(title_block
+		(title "SSD_XX_200_LPDRM")
+		(comment 1 "Vipul Singh")
+	)
+	(symbol
+		(lib_id "Non-Isolated-Buck-Module_v9:LPBM_tri_rail")
+		(at 133.35 71.12 0)
+		(unit 1)
+		(exclude_from_sim no)
+		(in_bom yes)
+		(on_board yes)
+		(dnp no)
+		(fields_autoplaced yes)
+		(property "Reference" "U8"
+			(at 133.35 67.31 0)
+			(effects
+				(font
+					(size 1.27 1.27)
+				)
+			)
+		)
+		(property "Value" "~"
+			(at 133.35 69.85 0)
+			(effects
+				(font
+					(size 1.27 1.27)
+				)
+			)
+		)
+		(property "Footprint" ""
+			(at 133.35 71.12 0)
+			(effects
+				(font
+					(size 1.27 1.27)
+				)
+				(hide yes)
+			)
+		)
+		(property "Datasheet" ""
+			(at 133.35 71.12 0)
+			(effects
+				(font
+					(size 1.27 1.27)
+				)
+				(hide yes)
+			)
+		)
+		(property "Description" ""
+			(at 133.35 71.12 0)
+			(effects
+				(font
+					(size 1.27 1.27)
+				)
+				(hide yes)
+			)
+		)
+		(pin "10"
+		)
+		(pin "1"
+		)
+		(pin "5"
+		)
+		(pin "6"
+		)
+		(pin "14"
+		)
+		(pin "4"
+		)
+		(pin "2"
+		)
+		(pin "7"
+		)
+		(pin "3"
+		)
+		(pin "8"
+		)
+		(pin "9"
+		)
+		(pin "12"
+		)
+		(pin "13"
+		)
+		(pin "11"
+		)
+		(instances
+			(project "SSD_XX_200_LPDRM"
+				(path "/75cb77c3-5cc7-465d-8913-c3025f73381b/5b718872-8a3b-4915-bd10-0e9e5cf53dc3/c4b977dc-80e1-41fb-acc6-bac4f39350df"
+					(reference "U8")
+					(unit 1)
+				)
+			)
+		)
+	)
 )
