File: Subsheets/Power Section.kicad_sch (KiCad schematic)
At the start: 0 parts

Commit message: Schematic Update-1.1
Connections:
- no-connect marks 2 -> 0
Other:
- sheet 12V_HPBM_MAIN renamed 12V HPBM Main
- sheet 12V_HPBM_RED renamed 12V HPBM Redundant
- sheet 3V3_HPBM_MAIN renamed 3V3 HPBM Main
- sheet 3V3_HPBM_RED renamed 3V3 HPBM Redundant
- sheet 5V_HPBM_MAIN renamed 5V HPBM Main
- sheet 5V_HPBM_RED renamed 5V HPBM Redundant
- sheet LPBM_MAIN renamed LPBM Main
- sheet LPBM_RED renamed LPBM Redundant
- sheet 12V HPBM Main ports: added 3V3, 5V; removed none
- sheet 12V HPBM Redundant ports: added 3V3, 5V; removed none
- sheet 3V3 HPBM Main ports: added 3V3, 5V; removed none
- sheet 3V3 HPBM Redundant ports: added 3V3, 5V; removed none
- sheet 5V HPBM Main ports: added 3V3, 5V; removed none
- sheet 5V HPBM Redundant ports: added 3V3, 5V; removed none
- sheet LPBM Main ports: added none; removed 1V8_BUCK_EN, 1V8_BUCK_OUT, 1V8_BUCK_PG, 1V8_BUCK_VMON
- sheet LPBM Redundant ports: added none; removed 1V8_BUCK_EN, 1V8_BUCK_OUT, 1V8_BUCK_PG, 1V8_BUCK_VMON
