File: Subsheets/Power Section.kicad_sch (KiCad schematic)
At the start: 0 parts

Commit message: Schematic Update 1.2
Other:
- sheet 12V HPBM Main ports: added PWR_IMON, PWR_OUT, PWR_PG, PWR_TEMP, PWR_VMON; removed BUCK_IMON, BUCK_OUT, BUCK_PG, BUCK_TEMP, BUCK_VMON
- sheet 12V HPBM Redundant ports: added PWR_IMON, PWR_OUT, PWR_PG, PWR_TEMP, PWR_VMON; removed BUCK_IMON, BUCK_OUT, BUCK_PG, BUCK_TEMP, BUCK_VMON
- sheet 3V3 HPBM Main ports: added PWR_IMON, PWR_OUT, PWR_PG, PWR_TEMP, PWR_VMON; removed BUCK_IMON, BUCK_OUT, BUCK_PG, BUCK_TEMP, BUCK_VMON
- sheet 3V3 HPBM Redundant ports: added PWR_IMON, PWR_OUT, PWR_PG, PWR_TEMP, PWR_VMON; removed BUCK_IMON, BUCK_OUT, BUCK_PG, BUCK_TEMP, BUCK_VMON
- sheet 5V HPBM Main ports: added PWR_IMON, PWR_OUT, PWR_PG, PWR_TEMP, PWR_VMON; removed BUCK_IMON, BUCK_OUT, BUCK_PG, BUCK_TEMP, BUCK_VMON
- sheet 5V HPBM Redundant ports: added PWR_IMON, PWR_OUT, PWR_PG, PWR_TEMP, PWR_VMON; removed BUCK_IMON, BUCK_OUT, BUCK_PG, BUCK_TEMP, BUCK_VMON
