File: Subsheets/Protection & Measurement.kicad_sch (KiCad schematic)
At the start: 13 parts

Commit message: Schematic Update-1.1
Parts:
- added C47: 0.1uF_50V_0402, Pixxel_Capacitors:CAP0402, symbol Device:C_Small
Connections:
- net GND: now also C47.2
- net Vmon: now also C47.1
Other:
- note added: "--------------------------------------------------------- TELEMETRY NOTE: UNREGULATED BUS VOLTAGE SCALING --------------------------------------------------------- Divider Ratio: 1/28 (R_TOP = 270 kΩ, R_BOT_EQ = 10 kΩ) EXPECTED ADC PIN VOLTAGES: - 22V -> 0.786V at ADC - 60V -> 2.143V at ADC (Note: C47 is a low-impedance charge reservoir to satisfy the AD7490's fast sampling gulp without causing v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"
- note removed: "Rail Split"
- moved on the sheet: R136, R137, R138, TP61
