File: Subsheets/Protection & Measurement.kicad_sch (KiCad schematic)
At the start: 14 parts

Commit message: Schematic Update 1.2
Changed lines of the file:
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@@
 		)
 	)
-	(text "---------------------------------------------------------\nTELEMETRY NOTE: UNREGULATED BUS VOLTAGE SCALING\n---------------------------------------------------------\nDivider Ratio: 1/28 (R_TOP = 270 kΩ, R_BOT_EQ = 10 kΩ)\n\nEXPECTED ADC PIN VOLTAGES:\n- 22V -> 0.786V at ADC\n- 60V -> 2.143V at ADC\n\n(Note: C47 is a low-impedance charge reservoir to satisfy \n     the AD7490's fast sampling gulp without causing voltage droop. Place it closeto the ADC input. \n---------------------------------------------------------"
+	(text "---------------------------------------------------------\nTELEMETRY NOTE: UNREGULATED BUS VOLTAGE SCALING\n---------------------------------------------------------\nDivider Ratio: 1/28 (R_TOP = 270 kΩ, R_BOT_EQ = 10 kΩ)\n\nEXPECTED ADC PIN VOLTAGES:\n- 22V -> 0.786V at ADC\n- 60V -> 2.143V at ADC\n\n(Note: C47 is a low-impedance charge reservoir to satisfy \n     the AD7490's fast sampling gulp without causing voltage droop. Place it close to the ADC input. \n---------------------------------------------------------"
 		(exclude_from_sim no)
 		(at 88.138 133.35 0)
