File: Subsheets/Temperature Sensor.kicad_sch (KiCad schematic)
At the start: 20 parts, among them U56 TMP100, U57 TMP100, U58 TMP100

Commit message: Schematic Update-1.1
Parts:
- removed C42: 0.1uF_50V_0402, Pixxel_Capacitors:CAP0402, symbol Device:C_Small
- removed R121, R126, R130: 0R_0.063W_0402, symbol Device:R_Small_US
- removed R132: 10k_0.0625W_0402, symbol Device:R_Small_US
- added C33: 0.1uF_50V_0402, Pixxel_Capacitors:CAP0402, symbol Device:C_Small
- added R120, R124, R129: 0R_0.063W_0402, Pixxel_Resistors:RES0402, symbol Device:R_Small_US
- added R159: 10k_0.0625W_0603, Pixxel_Resistors:RES0603, symbol Device:R_Small_US
- C41, C43: Manufacturer_Part_Number GCM155R71H104KE02J -> (none); Price(INR) (none) -> 9.45; Vendor_Part_Number 490-14514-2-ND -> (none)
- R119, R123, R128: footprint (none) -> Pixxel_Resistors:RES0402; Manufacturer_Name Vishay Dale -> (none); Manufacturer_Part_Number CRCW04020000Z0ED -> (none); Power Dissipation (W) 0.063 -> (none); Price 9.32 -> (none); Price(INR) (none) -> 9.45; Vendor Part Number (none) -> 541-0.0JTR-ND
- R134: value 10k_0.0625W_0402 -> 10k_0.0625W_0603; footprint (none) -> Pixxel_Resistors:RES0603; Manufacturer Name (none) -> Vishay Dale; Manufacturer Part Number (none) -> TNPW060310K0BEEA; Price(INR) (none) -> 24.57; Temp_max (C) (none) -> 175; Temp_min (C) (none) -> -55; Vendor (none) -> Digikey; Vendor Part Number (none) -> TNP10.0KAATR-ND
Connections:
- net 3V3: now also C33.1, R159.2
- net GND: now also C33.2
- net I2C_SCL: now also R120.2, R124.2, R129.2
- net at TP51.1, U57.1 (SCL): now also R124.1
- net at TP49.1, U56.1 (SCL): now also R120.1
- net at TP53.1, U58.1 (SCL): now also R129.1
- net at U58.3 (ADD1): now also R159.1
