File: Subsheets/Right Backplane Connector.kicad_sch (KiCad schematic)
At the start: 1 part, among them J2 SEAF-40-01-X-10-X-RA-GP-X-X

Commit message: Schematic Update 1.2
Parts:
- removed J2: SEAF-40-01-X-10-X-RA-GP-X-X, SEAF-40-01-X-10-X-RA-GP-X-X:SAMTEC_SEAF-40-01-X-10-X-RA-GP-X-X, symbol SEAF-40-01-X-10-X-RA-GP-X-X:SEAF-40-01-X-10-X-RA-GP-X-X
