File: Subsheets/Switch Main.kicad_sch (KiCad schematic)
At the start: 160 parts

Commit message: Schematic Update 1.2
Parts:
- removed JP58, JP59, JP60: SolderJumper_2_Open, symbol Jumper:SolderJumper_2_Open
- removed R1, R10, R11, R12, R13, R14, R15, R16, R17, R18, R19, R2, R20, R22, R23, R26, R27, R3, R30, R31, R37, R38, R4, R41, R42, R45, R46, R5, R51, R52, R53, R54, R55, R56, R57, R58, R6, R7, R8, R9: 10k_0.0625W_0402, symbol Device:R_Small_US
- removed R701, R703, R705, R707, R709, R711, R713, R715, R717, R719: 1.24M_0.0625W_0402, Pixxel_Resistors:RES0402, symbol Device:R_Small_US
- removed R702, R704, R706, R708, R710, R712, R714, R716, R718, R720, R722, R724, R726, R728, R730, R732, R734, R736, R738, R740: 100k_0.0625W_0402, Pixxel_Resistors:RES0402, symbol Device:R_Small_US
- removed R721, R723, R725, R727, R729, R731, R733: 432k_0.0625W_0402, symbol Device:R_Small_US
- removed R735, R737, R739: 267k_0.0625W_0402, Pixxel_Resistors:RES0402, symbol Device:R_Small_US
- removed U1, U10, U11, U12, U13, U14, U15, U16, U17, U18, U19, U2, U20, U3, U4, U5, U6, U7, U8, U9: (no value), symbol HVSM_LVSM_v9:LVSM
- added JP121, JP122, JP123: SolderJumper_2_Open, symbol Jumper:SolderJumper_2_Open
- added R757, R758, R759, R760, R761, R762, R763, R764, R765, R766, R767, R768, R769, R770, R771, R772, R773, R774, R775, R776, R777, R778, R779, R780, R781, R782, R783, R784, R785, R786, R787, R788, R789, R790, R791, R792, R793, R794, R795, R796, R797, R798, R799, R800, R801, R802, R803, R804, R805, R806, R807, R808, R809, R810, R811, R812, R813, R814, R815, R816: 100k_0.0625W_0402, Pixxel_Resistors:RES0402, symbol Device:R_Small_US
Connections:
- net 12V_OUT_MAIN: now also JP121.1 (A)
- net 3V3_OUT_MAIN: now also JP123.1 (A)
- net 5V_OUT_MAIN: now also JP122.1 (A)
- net SW10_EN_MAIN: now also R780.1
- net SW10_FLT_MAIN: now also R781.1
- net SW10_PG_MAIN: now also R786.1
- net SW11_EN_MAIN: now also R787.1
- net SW11_FLT_MAIN: now also R788.1
- net SW11_PG_MAIN: now also R789.1
- net SW12_EN_MAIN: now also R790.1
- net SW12_FLT_MAIN: now also R791.1
- net SW12_PG_MAIN: now also R792.1
- net SW13_EN_MAIN: now also R793.1
- net SW13_FLT_MAIN: now also R794.1
- net SW13_PG_MAIN: now also R795.1
- net SW14_EN_MAIN: now also R796.1
- net SW14_FLT_MAIN: now also R797.1
- net SW14_PG_MAIN: now also R798.1
- net SW15_EN_MAIN: now also R799.1
- net SW15_FLT_MAIN: now also R800.1
- net SW15_PG_MAIN: now also R801.1
- net SW16_EN_MAIN: now also R802.1
- net SW16_FLT_MAIN: now also R803.1
- net SW16_PG_MAIN: now also R804.1
- net SW17_EN_MAIN: now also R805.1
- net SW17_FLT_MAIN: now also R806.1
- net SW17_PG_MAIN: now also R807.1
- net SW18_EN_MAIN: now also R808.1
- net SW18_FLT_MAIN: now also R809.1
- net SW18_PG_MAIN: now also R810.1
- net SW19_EN_MAIN: now also R811.1
- net SW19_FLT_MAIN: now also R812.1
- net SW19_PG_MAIN: now also R813.1
- net SW1_EN_MAIN: now also R757.1
- net SW1_FLT_MAIN: now also R758.1
- net SW1_PG_MAIN: now also R759.1
- net SW20_EN_MAIN: now also R814.1
- net SW20_FLT_MAIN: now also R815.1
- net SW20_PG_MAIN: now also R816.1
- net SW2_EN_MAIN: now also R760.1
- net SW2_FLT_MAIN: now also R761.1
- net SW2_PG_MAIN: now also R762.1
- net SW3_EN_MAIN: now also R763.1
- net SW3_FLT_MAIN: now also R764.1
- net SW3_PG_MAIN: now also R765.1
- net SW4_EN_MAIN: now also R766.1
- net SW4_FLT_MAIN: now also R767.1
- net SW4_PG_MAIN: now also R768.1
- net SW5_EN_MAIN: now also R769.1
- net SW5_FLT_MAIN: now also R770.1
- net SW5_PG_MAIN: now also R771.1
- net SW6_EN_MAIN: now also R772.1
- net SW6_FLT_MAIN: now also R773.1
- net SW6_PG_MAIN: now also R782.1
- net SW7_EN_MAIN: now also R774.1
- net SW7_FLT_MAIN: now also R775.1
- net SW7_PG_MAIN: now also R783.1
- net SW8_EN_MAIN: now also R776.1
- net SW8_FLT_MAIN: now also R777.1
- net SW8_PG_MAIN: now also R784.1
- net SW9_EN_MAIN: now also R778.1
- net SW9_FLT_MAIN: now also R779.1
- net SW9_PG_MAIN: now also R785.1
- net 3V3 LVSM SW6/IN: now reaches JP4.2 (B), JP5.2 (B), JP6.2 (B)
- net 3V3 LVSM SW6/IN: now also R772.2
- net 3V3 LVSM SW2/IN: now reaches JP13.2 (B), JP14.2 (B), JP15.2 (B)
- net 3V3 LVSM SW2/IN: now also R760.2
- net 12V LVSM SW18/IN: now reaches JP22.2 (B), JP23.2 (B), JP24.2 (B)
- net 12V LVSM SW18/IN: now also R808.2
- net 3V3 LVSM SW4/IN: now reaches JP37.2 (B), JP38.2 (B), JP39.2 (B)
- net 3V3 LVSM SW4/IN: now also R766.2
- net 5V LVSM SW14/IN: now reaches JP10.2 (B), JP11.2 (B), JP12.2 (B)
- net 5V LVSM SW14/IN: now also R796.2
- net 5V LVSM SW11/IN: now reaches JP7.2 (B), JP8.2 (B), JP9.2 (B)
- net 5V LVSM SW11/IN: now also R787.2
- net 12V LVSM SW20/IN: now reaches JP46.2 (B), JP47.2 (B), JP48.2 (B)
- net 12V LVSM SW20/IN: now also R814.2
- net 5V LVSM SW16/IN: now reaches JP55.2 (B), JP56.2 (B), JP57.2 (B)
- net 5V LVSM SW16/IN: now also R802.2
- net 3V3 LVSM SW7/IN: now reaches JP16.2 (B), JP17.2 (B), JP18.2 (B)
- net 3V3 LVSM SW7/IN: now also R774.2
- net 3V3 LVSM SW9/IN: now reaches JP40.2 (B), JP41.2 (B), JP42.2 (B)
- net 3V3 LVSM SW9/IN: now also R778.2
- net 3V3 LVSM SW5/IN: now reaches JP49.2 (B), JP50.2 (B), JP51.2 (B)
- net 3V3 LVSM SW5/IN: now also R769.2
- net 3V3 LVSM SW8/IN: now reaches JP28.2 (B), JP29.2 (B), JP30.2 (B)
- net 3V3 LVSM SW8/IN: now also R776.2
- net 5V LVSM SW13/IN: now reaches JP31.2 (B), JP32.2 (B), JP33.2 (B)
- net 5V LVSM SW13/IN: now also R793.2
- net 5V LVSM SW12/IN: now reaches JP19.2 (B), JP20.2 (B), JP21.2 (B)
- net 5V LVSM SW12/IN: now also R790.2
- net 3V3 LVSM SW10/IN: now reaches JP52.2 (B), JP53.2 (B), JP54.2 (B)
- net 3V3 LVSM SW10/IN: now also R780.2
- net 3V3 LVSM SW1/IN: now reaches JP1.2 (B), JP2.2 (B), JP3.2 (B)
- net 3V3 LVSM SW1/IN: now also R757.2
- net 12V LVSM SW19/IN: now reaches JP34.2 (B), JP35.2 (B), JP36.2 (B)
- net 12V LVSM SW19/IN: now also R811.2
- net 3V3 LVSM SW3/IN: now reaches JP25.2 (B), JP26.2 (B), JP27.2 (B)
- net 3V3 LVSM SW3/IN: now also R763.2
- net 5V LVSM SW15/IN: now reaches JP43.2 (B), JP44.2 (B), JP45.2 (B)
- net 5V LVSM SW15/IN: now also R799.2
- new net 3V3_MAIN: R758.2, R759.2, R761.2, R762.2, R764.2, R765.2, R767.2, R768.2, R770.2, R771.2, R773.2, R775.2, R777.2, R779.2, R781.2, R782.2, R783.2, R784.2, R785.2, R786.2, R788.2, R789.2, R791.2, R792.2, R794.2, R795.2, R797.2, R798.2, R800.2, R801.2, R803.2, R804.2, R806.2, R807.2, R809.2, R810.2, R812.2, R813.2, R815.2, R816.2
- new net 5V LVSM SW17/IN: JP121.2 (B), JP122.2 (B), JP123.2 (B), R805.2
Other:
- added sheet 12V LVSM SW18 (12V LVSM.kicad_sch)
- added sheet 12V LVSM SW19 (12V LVSM.kicad_sch)
- added sheet 12V LVSM SW20 (12V LVSM.kicad_sch)
- added sheet 3V3 LVSM SW1 (3V3 LVSM.kicad_sch)
- added sheet 3V3 LVSM SW10 (3V3 LVSM.kicad_sch)
- added sheet 3V3 LVSM SW2 (3V3 LVSM.kicad_sch)
- added sheet 3V3 LVSM SW3 (3V3 LVSM.kicad_sch)
- added sheet 3V3 LVSM SW4 (3V3 LVSM.kicad_sch)
- added sheet 3V3 LVSM SW5 (3V3 LVSM.kicad_sch)
- added sheet 3V3 LVSM SW6 (3V3 LVSM.kicad_sch)
- added sheet 3V3 LVSM SW7 (3V3 LVSM.kicad_sch)
- added sheet 3V3 LVSM SW8 (3V3 LVSM.kicad_sch)
- added sheet 3V3 LVSM SW9 (3V3 LVSM.kicad_sch)
- added sheet 5V LVSM SW11 (5V LVSM.kicad_sch)
- added sheet 5V LVSM SW12 (5V LVSM.kicad_sch)
- added sheet 5V LVSM SW13 (5V LVSM.kicad_sch)
- added sheet 5V LVSM SW14 (5V LVSM.kicad_sch)
- added sheet 5V LVSM SW15 (5V LVSM.kicad_sch)
- added sheet 5V LVSM SW16 (5V LVSM.kicad_sch)
- added sheet 5V LVSM SW17 (5V LVSM.kicad_sch)
- note removed: "Vovp = 0.99 x (1+ Rtop/Rbot)"
- note removed: "Vovp = 13.26V"
- note removed: "Vovp = 3.63V"
- note removed: "Vovp = 5.27V"
- moved on the sheet: JP1, JP2, JP3
