File: Subsheets/Switch Redundant.kicad_sch (KiCad schematic)
At the start: 120 parts

Commit message: Schematic Update 1.2
Parts:
- removed JP115, JP116, JP117, JP118, JP119, JP120: SolderJumper_2_Open, symbol Jumper:SolderJumper_2_Open
- removed R100, R101, R102, R59, R60, R61, R62, R63, R64, R65, R66, R67, R68, R69, R70, R75, R76, R77, R78, R79, R80, R81, R82, R83, R84, R85, R86, R87, R88, R89, R90, R91, R92, R93, R94, R95, R96, R97, R98, R99: 10k_0.0625W_0402, symbol Device:R_Small_US
- removed U29, U30, U31, U32, U33, U34, U35, U36, U37, U38, U39, U40, U41, U42, U43, U44, U45, U46, U47, U48: (no value), symbol HVSM_LVSM_v9:LVSM
- added JP124, JP125, JP126, JP58, JP59, JP60: SolderJumper_2_Open, symbol Jumper:SolderJumper_2_Open
- added R817, R818, R819, R820, R821, R822, R823, R824, R825, R826, R827, R828, R829, R830, R831, R832, R833, R834, R835, R836, R837, R838, R839, R840, R841, R842, R843, R844, R845, R846, R847, R848, R849, R850, R851, R852, R853, R854, R855, R856, R857, R858, R859, R860, R861, R862, R863, R864, R865, R866, R867, R868, R869, R870, R871, R872, R873, R874, R875, R876: 100k_0.0625W_0402, Pixxel_Resistors:RES0402, symbol Device:R_Small_US
Connections:
- net SW10_EN_RED: now also R840.1
- net SW10_FLT_RED: now also R841.1
- net SW10_PG_RED: now also R846.1
- net SW11_EN_RED: now also R847.1
- net SW11_FLT_RED: now also R848.1
- net SW11_PG_RED: now also R851.1
- net SW12_EN_RED: now also R858.1
- net SW12_FLT_RED: now also R859.1
- net SW12_PG_RED: now also R865.1
- net SW13_EN_RED: now also R871.1
- net SW13_FLT_RED: now also R872.1
- net SW13_PG_RED: now also R875.1
- net SW14_EN_RED: now also R849.1
- net SW14_FLT_RED: now also R850.1
- net SW14_PG_RED: now also R852.1
- net SW15_EN_RED: now also R860.1
- net SW15_FLT_RED: now also R861.1
- net SW15_PG_RED: now also R866.1
- net SW16_EN_RED: now also R873.1
- net SW16_FLT_RED: now also R874.1
- net SW16_PG_RED: now also R876.1
- net SW17_EN_RED: now also R862.1
- net SW17_FLT_RED: now also R863.1
- net SW17_PG_RED: now also R867.1
- net SW18_EN_RED: now also R853.1
- net SW18_FLT_RED: now also R854.1
- net SW18_PG_RED: now also R855.1
- net SW19_EN_RED: now also R868.1
- net SW19_FLT_RED: now also R869.1
- net SW19_PG_RED: now also R870.1
- net SW1_EN_RED: now also R817.1
- net SW1_FLT_RED: now also R818.1
- net SW1_PG_RED: now also R827.1
- net SW20_EN_RED: now also R856.1
- net SW20_FLT_RED: now also R857.1
- net SW20_PG_RED: now also R864.1
- net SW2_EN_RED: now also R819.1
- net SW2_FLT_RED: now also R820.1
- net SW2_PG_RED: now also R828.1
- net SW3_EN_RED: now also R821.1
- net SW3_FLT_RED: now also R822.1
- net SW3_PG_RED: now also R829.1
- net SW4_EN_RED: now also R823.1
- net SW4_FLT_RED: now also R824.1
- net SW4_PG_RED: now also R830.1
- net SW5_EN_RED: now also R825.1
- net SW5_FLT_RED: now also R826.1
- net SW5_PG_RED: now also R831.1
- net SW6_EN_RED: now also R832.1
- net SW6_FLT_RED: now also R833.1
- net SW6_PG_RED: now also R842.1
- net SW7_EN_RED: now also R834.1
- net SW7_FLT_RED: now also R835.1
- net SW7_PG_RED: now also R843.1
- net SW8_EN_RED: now also R836.1
- net SW8_FLT_RED: now also R837.1
- net SW8_PG_RED: now also R844.1
- net SW9_EN_RED: now also R838.1
- net SW9_FLT_RED: now also R839.1
- net SW9_PG_RED: now also R845.1
- net 5V LVSM SW13/IN: now reaches JP109.2 (B), JP110.2 (B), JP111.2 (B)
- net 5V LVSM SW13/IN: now also R871.2
- net 3V3 LVSM SW6/IN: now reaches JP73.2 (B), JP74.2 (B), JP75.2 (B)
- net 3V3 LVSM SW6/IN: now also R832.2
- net 3V3 LVSM SW10/IN: now reaches JP85.2 (B), JP86.2 (B), JP87.2 (B)
- net 3V3 LVSM SW10/IN: now also R840.2
- net 3V3 LVSM SW3/IN: now reaches JP64.2 (B), JP65.2 (B), JP66.2 (B)
- net 3V3 LVSM SW3/IN: now also R821.2
- net 3V3 LVSM SW8/IN: now reaches JP79.2 (B), JP80.2 (B), JP81.2 (B)
- net 3V3 LVSM SW8/IN: now also R836.2
- net 5V LVSM SW16/IN: now reaches JP112.2 (B), JP113.2 (B), JP114.2 (B)
- net 5V LVSM SW16/IN: now also R873.2
- net 5V LVSM SW15/IN: now reaches JP103.2 (B), JP104.2 (B), JP105.2 (B)
- net 5V LVSM SW15/IN: now also R860.2
- net 3V3 LVSM SW2/IN: now reaches JP61.2 (B), JP62.2 (B), JP63.2 (B)
- net 3V3 LVSM SW2/IN: now also R819.2
- net 3V3 LVSM SW4/IN: now reaches JP67.2 (B), JP68.2 (B), JP69.2 (B)
- net 3V3 LVSM SW4/IN: now also R823.2
- net 12V LVSM SW19/IN: now reaches JP106.2 (B), JP107.2 (B), JP108.2 (B)
- net 12V LVSM SW19/IN: now also R868.2
- net 12V LVSM SW20/IN: now reaches JP97.2 (B), JP98.2 (B), JP99.2 (B)
- net 12V LVSM SW20/IN: now also R856.2
- net 3V3 LVSM SW5/IN: now reaches JP70.2 (B), JP71.2 (B), JP72.2 (B)
- net 3V3 LVSM SW5/IN: now also R825.2
- net 5V LVSM SW12/IN: now reaches JP100.2 (B), JP101.2 (B), JP102.2 (B)
- net 5V LVSM SW12/IN: now also R858.2
- net 12V LVSM SW18/IN: now reaches JP94.2 (B), JP95.2 (B), JP96.2 (B)
- net 12V LVSM SW18/IN: now also R853.2
- net 5V LVSM SW14/IN: now reaches JP91.2 (B), JP92.2 (B), JP93.2 (B)
- net 5V LVSM SW14/IN: now also R849.2
- net 5V LVSM SW11/IN: now reaches JP88.2 (B), JP89.2 (B), JP90.2 (B)
- net 5V LVSM SW11/IN: now also R847.2
- net 3V3 LVSM SW7/IN: now reaches JP76.2 (B), JP77.2 (B), JP78.2 (B)
- net 3V3 LVSM SW7/IN: now also R834.2
- net 3V3 LVSM SW9/IN: now reaches JP82.2 (B), JP83.2 (B), JP84.2 (B)
- net 3V3 LVSM SW9/IN: now also R838.2
- net 12V_OUT_RED renamed 12V_OUT_MAIN
- net 12V_OUT_MAIN: now also JP124.1 (A), JP58.1 (A)
- net 3V3_OUT_RED renamed 3V3_OUT_MAIN
- net 3V3_OUT_MAIN: now also JP126.1 (A), JP60.1 (A)
- net 5V_OUT_RED renamed 5V_OUT_MAIN
- net 5V_OUT_MAIN: now also JP125.1 (A), JP59.1 (A)
- new net 3V3 LVSM SW1/IN: JP58.2 (B), JP59.2 (B), JP60.2 (B), R817.2
- new net 3V3_RED: R818.2, R820.2, R822.2, R824.2, R826.2, R827.2, R828.2, R829.2, R830.2, R831.2, R833.2, R835.2, R837.2, R839.2, R841.2, R842.2, R843.2, R844.2, R845.2, R846.2, R848.2, R850.2, R851.2, R852.2, R854.2, R855.2, R857.2, R859.2, R861.2, R863.2, R864.2, R865.2, R866.2, R867.2, R869.2, R870.2, R872.2, R874.2, R875.2, R876.2
- new net 5V LVSM SW17/IN: JP124.2 (B), JP125.2 (B), JP126.2 (B), R862.2
Other:
- added sheet 12V LVSM SW18 (12V LVSM.kicad_sch)
- added sheet 12V LVSM SW19 (12V LVSM.kicad_sch)
- added sheet 12V LVSM SW20 (12V LVSM.kicad_sch)
- added sheet 3V3 LVSM SW1 (3V3 LVSM.kicad_sch)
- added sheet 3V3 LVSM SW10 (3V3 LVSM.kicad_sch)
- added sheet 3V3 LVSM SW2 (3V3 LVSM.kicad_sch)
- added sheet 3V3 LVSM SW3 (3V3 LVSM.kicad_sch)
- added sheet 3V3 LVSM SW4 (3V3 LVSM.kicad_sch)
- added sheet 3V3 LVSM SW5 (3V3 LVSM.kicad_sch)
- added sheet 3V3 LVSM SW6 (3V3 LVSM.kicad_sch)
- added sheet 3V3 LVSM SW7 (3V3 LVSM.kicad_sch)
- added sheet 3V3 LVSM SW8 (3V3 LVSM.kicad_sch)
- added sheet 3V3 LVSM SW9 (3V3 LVSM.kicad_sch)
- added sheet 5V LVSM SW11 (5V LVSM.kicad_sch)
- added sheet 5V LVSM SW12 (5V LVSM.kicad_sch)
- added sheet 5V LVSM SW13 (5V LVSM.kicad_sch)
- added sheet 5V LVSM SW14 (5V LVSM.kicad_sch)
- added sheet 5V LVSM SW15 (5V LVSM.kicad_sch)
- added sheet 5V LVSM SW16 (5V LVSM.kicad_sch)
- added sheet 5V LVSM SW17 (5V LVSM.kicad_sch)
- note added: "12V SWITCHES"
- note added: "3V3 SWITCHES"
- note added: "5V SWITCHES"
