File: Subshhets/IO Expander.kicad_sch (KiCad schematic)
At the start: 27 parts, among them U50 MCP23017_ML, U52 MCP23017_ML, U54 MCP23017_ML

Commit message: Schematic Update-1.1
Parts:
- removed C33: 0.1uF_50V_0402, Pixxel_Capacitors:CAP0402, symbol Device:C_Small
- added C55: 0.1uF_50V_0402, Pixxel_Capacitors:CAP0402, symbol Device:C_Small
- C29, C37: Manufacturer_Part_Number GCM155R71H104KE02J -> (none); Price(INR) (none) -> 9.45; Vendor_Part_Number 490-14514-2-ND -> (none)
- C30, C34, C38: footprint (none) -> Pixxel_Capacitors:CAP0805; Manufacturer Murata Electronics -> (none); Manufacturer Name (none) -> Murata Electronics; Manufacturer_Part_Number GCM21BR71A106KE22L -> (none); Mass (grams) 0.001 -> (none); Power Dissipation (W) NA -> (none); Price(INR) (none) -> 34.97; RQjC (C/W) NA -> (none); Temp_max (C) 105 -> 125; Vendor (none) -> Digikey; Vendor Part Number (none) -> 490-10674-2-ND
- R103, R107, R108, R113, R114, R125: footprint (none) -> Pixxel_Resistors:RES0402; Manufacturer_Name Vishay Dale -> (none); Manufacturer_Part_Number CRCW04020000Z0ED -> (none); Power Dissipation (W) 0.063 -> (none); Price 9.32 -> (none); Price(INR) (none) -> 9.45; Vendor Part Number (none) -> 541-0.0JTR-ND
- R105: value 10k_0.0625W_0402 -> 10k_0.0625W_0603; footprint Pixxel_Resistors:RES0402 -> Pixxel_Resistors:RES0603; Manufacturer Name (none) -> Vishay Dale; Manufacturer Part Number (none) -> TNPW060310K0BEEA; Price(INR) (none) -> 24.57; Temp_max (C) (none) -> 175; Temp_min (C) (none) -> -55; Vendor (none) -> Digikey; Vendor Part Number (none) -> TNP10.0KAATR-ND
- R109, R115: value 10k_0.0625W_0402 -> 10k_0.0625W_0603; footprint (none) -> Pixxel_Resistors:RES0603; Manufacturer Name (none) -> Vishay Dale; Manufacturer Part Number (none) -> TNPW060310K0BEEA; Price(INR) (none) -> 24.57; Temp_max (C) (none) -> 175; Temp_min (C) (none) -> -55; Vendor (none) -> Digikey; Vendor Part Number (none) -> TNP10.0KAATR-ND
Connections:
- net 3V3: now also C55.1
- net GND: now also C55.2
