File: Subshhets/GPIO Expanders.kicad_sch (KiCad schematic)
At the start: 0 parts

Commit message: Schematic Update 1.2
Other:
- note added: "IO Bank-1"
- note added: "IO Bank-2"
- note added: "IO Bank-3"
Changed lines of the file:
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@@
 		(comment 1 "Vipul Singh")
+	)
+	(text "IO Bank-3"
+		(exclude_from_sim no)
+		(at 201.93 132.588 0)
+		(effects
+			(font
+				(size 1.905 1.905)
+				(thickness 0.381)
+				(bold yes)
+			)
+		)
+	)
+	(text "IO Bank-2"
+		(exclude_from_sim no)
+		(at 202.438 100.33 0)
+		(effects
+			(font
+				(size 1.905 1.905)
+				(thickness 0.381)
+				(bold yes)
+			)
+		)
+	)
+	(text "IO Bank-3"
+		(exclude_from_sim no)
+		(at 81.026 131.572 0)
+		(effects
+			(font
+				(size 1.905 1.905)
+				(thickness 0.381)
+				(bold yes)
+			)
+		)
+	)
+	(text "IO Bank-1"
+		(exclude_from_sim no)
+		(at 81.28 65.786 0)
+		(effects
+			(font
+				(size 1.905 1.905)
+				(thickness 0.381)
+				(bold yes)
+			)
+		)
+	)
+	(text "IO Bank-2"
+		(exclude_from_sim no)
+		(at 81.534 99.314 0)
+		(effects
+			(font
+				(size 1.905 1.905)
+				(thickness 0.381)
+				(bold yes)
+			)
+		)
+	)
+	(text "IO Bank-1"
+		(exclude_from_sim no)
+		(at 202.184 66.802 0)
+		(effects
+			(font
+				(size 1.905 1.905)
+				(thickness 0.381)
+				(bold yes)
+			)
+		)
 	)
 	(no_connect
@@
 		)
 	)
+	(polyline
+		(pts
+			(xy 57.15 81.28) (xy 105.41 81.28)
+		)
+		(stroke
+			(width 0.254)
+			(type dash)
+		)
+	)
 	(wire
 		(pts
@@
 		)
 	)
+	(polyline
+		(pts
+			(xy 177.8 114.3) (xy 226.06 114.3)
+		)
+		(stroke
+			(width 0.254)
+			(type dash)
+		)
+	)
 	(wire
 		(pts
@@
 		)
 	)
+	(polyline
+		(pts
+			(xy 177.8 48.26) (xy 226.06 48.26)
+		)
+		(stroke
+			(width 0.254)
+			(type dash)
+		)
+	)
 	(wire
 		(pts
@@
 		)
 	)
+	(polyline
+		(pts
+			(xy 57.15 46.99) (xy 105.41 46.99)
+		)
+		(stroke
+			(width 0.254)
+			(type dash)
+		)
+	)
 	(wire
 		(pts
@@
 		)
 	)
+	(polyline
+		(pts
+			(xy 177.8 81.28) (xy 226.06 81.28)
+		)
+		(stroke
+			(width 0.254)
+			(type dash)
+		)
+	)
 	(wire
 		(pts
@@
 		)
 	)
+	(polyline
+		(pts
+			(xy 57.15 114.3) (xy 105.41 114.3)
+		)
+		(stroke
+			(width 0.254)
+			(type dash)
+		)
+	)
